Commit message: Added event classification

File: robot_tppo/urdf/camera.urdf.xacro (robot description, xacro)
@@ -3,5 +3,5 @@
       <!-- STEP 7 - Camera -->
     <joint type="fixed" name="camera_joint">
-        <origin xyz="0.225 0 0.075" rpy="0 0 0"/>
+        <origin xyz="0.0 0 0.075" rpy="0 0 0"/>
         <child link="camera_link"/>
         <parent link="base_link"/>

File: robot_tppo/urdf/lidar.urdf.xacro (robot description, xacro)
@@ -29,5 +29,5 @@
       </geometry>
     </visual-->
-</link>
+	</link>
   <gazebo reference="scan_link">
     <sensor name="gpu_lidar" type="gpu_lidar">

File: robot_tppo/urdf/robot.urdf.xacro (robot description, xacro)
@@ -5,4 +5,5 @@
     <xacro:include filename="lidar.urdf.xacro"/>
     <xacro:include filename="inertial_measuring_unit.urdf.xacro"/>
+    <xacro:include filename="odometry.urdf.xacro"/>
     <ros2_control name="my_robot_hardware" type="system">
         <hardware>
